File: Hardware/PCB/Suntracker/Suntracker.kicad_pcb (KiCad board)
At the start: 2 copper layers, 104 x 76 mm, 113 parts, among them J1 FotoPanel_IN, J10 STM_3.3V_PROG, J11 STM_NRST, J12 STM_BOOT, J13 MOTOR_1+, J14 MOTOR_1-, J15 MOTOR_2+, J16 MOTOR_2-, J17 STM_GND_PROG, J18 SERVO_1_SIGNAL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

Commit message: Cleaning be4 final documentation
Parts:
- added G***: LOGO, PCB:logo_bs, F.Cu at (177.0, 72.5)
- added G***: LOGO, PCB:Logo, B.Cu at (170.5, 71.7)
